File: maester_tarly.kicad_pcb (KiCad board)
At the start: 4 copper layers, 72 x 62.4 mm, 126 parts, among them J101 Micro_SD_Card_Det, J102 USB_B_Micro, J103 USB_A, J104 Conn_01x06, J105 Conn_01x10, J106 RJ45_Amphenol_RJMG1BD3B8K1ANR, J107 DF40GB(1.5)-48DS-0.4V, J108 DF40GB(1.5)-48DS-0.4V, J109 DF40GB(1.5)-48DS-0.4V, J110 DF40GB(1.5)-48DS-0.4V, U1 SAM9X60, U2 W971GG6SB-18, U3 MCP16501, U501 KSZ8081RNA, Y401 32.768kHz, Y402 DSC1001, Y501 DSC1001

Commit message: Redid all the wiggle-wiggles
Routing:
- net /CPU_CORE/data6: track 26.8 -> 44.0 mm
- net /CPU_CORE/data9: track 26.9 -> 44.0 mm
- net /CPU_CORE/CPU_DDR_LOW_MASK: track 28.7 -> 44.5 mm
- net /CPU_CORE/addr12: track 31.2 -> 44.0 mm
- net /CPU_CORE/addr7: track 34.3 -> 44.0 mm
- net /CPU_CORE/addr5: track 32.2 -> 40.0 mm
- net /CPU_CORE/addr10: track 36.3 -> 44.0 mm
- net /CPU_CORE/data14: track 36.7 -> 44.0 mm
- net /CPU_CORE/addr1: track 36.9 -> 44.0 mm
- net /CPU_CORE/addr3: track 37.0 -> 44.0 mm
- net /CPU_CORE/data1: track 38.1 -> 44.4 mm
- net /CPU_CORE/data8: track 37.9 -> 44.0 mm
- net /CPU_CORE/CPU_DDR_HIGH_STROBE_P: track 38.9 -> 44.3 mm
- net /CPU_CORE/data0: track 38.7 -> 44.0 mm
- net /CPU_CORE/data15: track 39.0 -> 44.1 mm
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
Commit message: Clean DRC
Parts:
- moved C416 0.39 mm to (123.4, 141.2)
Routing:
- net +5V: track 139.4 -> 121.9 mm
- net /CPU_IO/PHY_TXD0: track 12.0 -> 8.97 mm
- net +3V3: track 56.8 -> 57.8 mm
- net /a21: track 42.9 -> 42.3 mm
- net GND: track 216.6 -> 216.0 mm
